File: CAN Bus Organizer 8/CAN Bus Organizer.kicad_pcb (KiCad board)
At the start: 2 copper layers, 212 x 10 mm, 20 parts, among them J1 Conn_01x02_Male, J10 Conn_01x02_Male, J11 Conn_01x02_Male, J12 Conn_01x02_Male, J13 Conn_01x02_Male, J14 Conn_01x02_Male, J15 Conn_01x02_Male, J16 Conn_01x02_Male, J17 Conn_01x02_Male, J18 Conn_01x02_Male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

Commit message: Finished board layout
Routing:
- net Net-(J17-Pad2): track 0.00 -> 12.3 mm
- net Net-(J12-Pad2): track 0.00 -> 12.3 mm
- net Net-(J18-Pad2): track 0.00 -> 12.3 mm
- net Net-(J16-Pad2): track 0.00 -> 12.3 mm
- net Net-(J15-Pad2): track 0.00 -> 12.3 mm
- net Net-(J14-Pad2): track 0.00 -> 12.3 mm
- net Net-(J13-Pad2): track 0.00 -> 12.3 mm
- net Net-(J11-Pad2): track 0.00 -> 12.3 mm
- net Net-(J1-Pad2): track 0.00 -> 12.3 mm
- net Net-(J18-Pad1): track 0.00 -> 12.0 mm
- net Net-(J17-Pad1): track 0.00 -> 12.0 mm
- net Net-(J16-Pad1): track 0.00 -> 12.0 mm
- net Net-(J15-Pad1): track 0.00 -> 12.0 mm
- net Net-(J14-Pad1): track 0.00 -> 12.0 mm
- net Net-(J13-Pad1): track 0.00 -> 12.0 mm
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Other:
- net class Default: trace_width 0.25 -> 1
- rule pad_to_mask_clearance: 0.2 -> 0
- board text added: "Can Bus Organizer 12 Rev 1 Corwin Hansen"
Changed lines of the file:
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@@
   (general
     (thickness 1.6)
-    (drawings 4)
-    (tracks 0)
+    (drawings 5)
+    (tracks 55)
     (zones 0)
     (modules 20)
@@
   )
   (setup
-    (last_trace_width 0.25)
+    (last_trace_width 1)
     (trace_clearance 0.2)
     (zone_clearance 0.508)
@@
     (pad_size 1.524 1.524)
     (pad_drill 0.762)
-    (pad_to_mask_clearance 0.2)
+    (pad_to_mask_clearance 0)
     (aux_axis_origin 0 0)
     (visible_elements FFFFFF7F)
@@
       (drillshape 0)
       (scaleselection 1)
-      (outputdirectory "../../CAN Bus Organizer 8 Gerber/"))
+      (outputdirectory "../CAN Bus Organizer 8 Gerber/"))
   )
   (net 0 "")
@@
   (net_class Default "This is the default net class."
     (clearance 0.2)
-    (trace_width 0.25)
+    (trace_width 1)
     (via_dia 0.8)
     (via_drill 0.4)
@@
     (pad 1 np_thru_hole circle (at 0 0) (size 4.3 4.3) (drill 4.3) (layers *.Cu *.Mask))
   )
+  (gr_text "Can Bus Organizer 12   Rev 1   Corwin Hansen" (at 136 71) (layer B.SilkS)
+    (effects (font (size 1.5 1.5) (thickness 0.3)) (justify mirror))
+  )
   (gr_line (start 242 63) (end 30 63) (layer Edge.Cuts) (width 0.2))
   (gr_line (start 242 73) (end 242 63) (layer Edge.Cuts) (width 0.2))
   (gr_line (start 30 73) (end 242 73) (layer Edge.Cuts) (width 0.2))
   (gr_line (start 30 63) (end 30 73) (layer Edge.Cuts) (width 0.2))
+  (segment (start 46 69) (end 58 69) (width 1) (layer F.Cu) (net 1))
+  (segment (start 46 66) (end 48.089998 66) (width 1) (layer F.Cu) (net 2))
+  (segment (start 48.089998 66) (end 48.399999 66.310001) (width 1) (layer F.Cu) (net 2))
+  (segment (start 48.399999 66.310001) (end 56.558629 66.310001) (width 1) (layer F.Cu) (net 2))
+  (segment (start 56.558629 66.310001) (end 56.86863 66) (width 1) (layer F.Cu) (net 2))
+  (segment (start 56.86863 66) (end 58 66) (width 1) (layer F.Cu) (net 2))
+  (segment (start 67 66) (end 69.089998 66) (width 1) (layer F.Cu) (net 3))
+  (segment (start 69.089998 66) (end 69.399999 66.310001) (width 1) (layer F.Cu) (net 3))
+  (segment (start 69.399999 66.310001) (end 77.558629 66.310001) (width 1) (layer F.Cu) (net 3))
+  (segment (start 77.558629 66.310001) (end 77.86863 66) (width 1) (layer F.Cu) (net 3))
+  (segment (start 77.86863 66) (end 79 66) (width 1) (layer F.Cu) (net 3))
+  (segment (start 67 69) (end 79 69) (width 1) (layer F.Cu) (net 4))
+  (segment (start 88 66) (end 90.089998 66) (width 1) (layer F.Cu) (net 5))
+  (segment (start 90.399999 66.310001) (end 98.558629 66.310001) (width 1) (layer F.Cu) (net 5))
+  (segment (start 90.089998 66) (end 90.399999 66.310001) (width 1) (layer F.Cu) (net 5))
+  (segment (start 98.558629 66.310001) (end 98.86863 66) (width 1) (layer F.Cu) (net 5))
+  (segment (start 98.86863 66) (end 100 66) (width 1) (layer F.Cu) (net 5))
+  (segment (start 88 69) (end 100 69) (width 1) (layer F.Cu) (net 6))
+  (segment (start 109 66) (end 111.089998 66) (width 1) (layer F.Cu) (net 7))
+  (segment (start 111.089998 66) (end 111.399999 66.310001) (width 1) (layer F.Cu) (net 7))
+  (segment (start 111.399999 66.310001) (end 119.558629 66.310001) (width 1) (layer F.Cu) (net 7))
+  (segment (start 119.558629 66.310001) (end 119.86863 66) (width 1) (layer F.Cu) (net 7))
+  (segment (start 119.86863 66) (end 121 66) (width 1) (layer F.Cu) (net 7))
+  (segment (start 109 69) (end 121 69) (width 1) (layer F.Cu) (net 8))
+  (segment (start 130 66) (end 132.089998 66) (width 1) (layer F.Cu) (net 9))
+  (segment (start 132.089998 66) (end 132.399999 66.310001) (width 1) (layer F.Cu) (net 9))
+  (segment (start 140.558629 66.310001) (end 140.86863 66) (width 1) (layer F.Cu) (net 9))
+  (segment (start 140.86863 66) (end 141.96863 66) (width 1) (layer F.Cu) (net 9))
+  (segment (start 132.399999 66.310001) (end 140.558629 66.310001) (width 1) (layer F.Cu) (net 9))
+  (segment (start 141.96863 66) (end 142 66) (width 1) (layer F.Cu) (net 9))
+  (segment (start 130 69) (end 142 69) (width 1) (layer F.Cu) (net 10))
+  (segment (start 163 66) (end 161.86863 66) (width 1) (layer F.Cu) (net 11))
+  (segment (start 161.86863 66) (end 161.558629 66.310001) (width 1) (layer F.Cu) (net 11))
+  (segment (start 161.558629 66.310001) (end 153.399999 66.310001) (width 1) (layer F.Cu) (net 11))
+  (segment (start 153.399999 66.310001) (end 153.089998 66) (width 1) (layer F.Cu) (net 11))
+  (segment (start 153.089998 66) (end 151 66) (width 1) (layer F.Cu) (net 11))
+  (segment (start 151 69) (end 163 69) (width 1) (layer F.Cu) (net 12))
+  (segment (start 172 66) (end 174.089998 66) (width 1) (layer F.Cu) (net 13))
+  (segment (start 174.089998 66) (end 174.399999 66.310001) (width 1) (layer F.Cu) (net 13))
+  (segment (start 174.399999 66.310001) (end 182.558629 66.310001) (width 1) (layer F.Cu) (net 13))
+  (segment (start 182.558629 66.310001) (end 182.86863 66) (width 1) (layer F.Cu) (net 13))
+  (segment (start 182.86863 66) (end 184 66) (width 1) (layer F.Cu) (net 13))
+  (segment (start 172 69) (end 184 69) (width 1) (layer F.Cu) (net 14))
+  (segment (start 193 66) (end 195.089998 66) (width 1) (layer F.Cu) (net 15))
+  (segment (start 195.399999 66.310001) (end 203.558629 66.310001) (width 1) (layer F.Cu) (net 15))
+  (segment (start 195.089998 66) (end 195.399999 66.310001) (width 1) (layer F.Cu) (net 15))
+  (segment (start 203.558629 66.310001) (end 203.86863 66) (width 1) (layer F.Cu) (net 15))
+  (segment (start 203.86863 66) (end 205 66) (width 1) (layer F.Cu) (net 15))
+  (segment (start 193 69) (end 205 69) (width 1) (layer F.Cu) (net 16))
+  (segment (start 214 66) (end 216.089998 66) (width 1) (layer F.Cu) (net 17))
+  (segment (start 216.089998 66) (end 216.399999 66.310001) (width 1) (layer F.Cu) (net 17))
+  (segment (start 216.399999 66.310001) (end 224.558629 66.310001) (width 1) (layer F.Cu) (net 17))
+  (segment (start 224.558629 66.310001) (end 224.86863 66) (width 1) (layer F.Cu) (net 17))
+  (segment (start 224.86863 66) (end 226 66) (width 1) (layer F.Cu) (net 17))
+  (segment (start 214 69) (end 226 69) (width 1) (layer F.Cu) (net 18))
 )

Commit message: Changed board name
Other:
- board text added: "Can Bus Organizer 8 Rev 1 Corwin Hansen"
- board text removed: "Can Bus Organizer 12 Rev 1 Corwin Hansen"
Changed lines of the file:
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@@
     (pad 1 np_thru_hole circle (at 0 0) (size 4.3 4.3) (drill 4.3) (layers *.Cu *.Mask))
   )
-  (gr_text "Can Bus Organizer 12   Rev 1   Corwin Hansen" (at 136 71) (layer B.SilkS)
+  (gr_text "Can Bus Organizer 8   Rev 1   Corwin Hansen" (at 136 71) (layer B.SilkS)
     (effects (font (size 1.5 1.5) (thickness 0.3)) (justify mirror))
   )
